Commit message: Added state_publisher to omni_state.launch. Base link renamed into base_link.

File: omni_description/urdf/omni.urdf (robot description, URDF)
Before this commit: robot phantom_omni, 7 links, 6 joints
Links:
- removed link base
- added link base_link; visual mesh filename=package://omni_description/meshes/base.stl
Joints:
- joint waist: parent base -> base_link
