Commit message: Description parametrized (urdf -> xacro). Changed behaviors of buttons. Publishing current velocity.

File: omni_description/urdf/omni.urdf.xacro (robot description, xacro)
@@ -1,4 +1,5 @@
 <?xml version="1.0" encoding="utf-8"?>
 <robot name="phantom_omni" xmlns:xacro="http://www.ros.org/wiki/xacro">
+  <property name="pi" value="3.1415926535897931" />
 	<!-- Materials -->
 	<material name="metal_seamed">
@@ -12,7 +13,9 @@
 	</material>
 	<!-- Links -->
+  <link name="base" >
+  </link>
   <link name="base_link" >
     <visual>
-			<origin xyz="0 -0.02 0" />
+      <origin xyz="0 -0.02 0" rpy="0 0 0" />
       <geometry>
 				<mesh filename="package://omni_description/meshes/base.stl" />
@@ -23,5 +26,5 @@
   <link name="torso" >
     <visual>
-			<origin xyz="0 0 0.036" rpy="-1.5707 0 0"/>
+      <origin xyz="0 0 0.036" rpy="${-pi/2} 0 0"/>
       <geometry>
 				<mesh filename="package://omni_description/meshes/torso.stl" />
@@ -41,5 +44,5 @@
   <link name="lower_arm" >
 		<visual>
-			<origin xyz="0 0 0" rpy="1.5707 0 0"/>
+      <origin xyz="0 0 0" rpy="${pi/2} 0 0"/>
       <geometry>
 				<mesh filename="package://omni_description/meshes/lower_arm.stl" />
@@ -50,5 +53,5 @@
   <link name="wrist" >
 		<visual>
-			<origin xyz="0 0 0" rpy="3.14159 0 0"/>
+      <origin xyz="0 0 0" rpy="${pi} 0 0"/>
       <geometry>
 				<mesh filename="package://omni_description/meshes/wrist.stl" />
@@ -59,5 +62,5 @@
   <link name="tip" >
 		<visual>
-			<origin xyz="0 0 0" rpy="-1.5707 0 0"/>
+      <origin xyz="0 0 0" rpy="${-pi/2} 0 0"/>
       <geometry>
 				<mesh filename="package://omni_description/meshes/tip.stl" />
@@ -68,5 +71,5 @@
   <link name="stylus" >
     <visual>
-			<origin xyz="0 -0.033 0" rpy="1.5707 1.5707 0"/>
+      <origin xyz="0 -0.033 0" rpy="${pi/2} ${pi/2} 0"/>
       <geometry>
 				<mesh filename="package://omni_description/meshes/pen.stl" />
@@ -76,4 +79,10 @@
   </link>
 	<!-- joints -->
+  <joint name="ref_base" type="fixed" >
+    <parent link="base" />
+    <child link="base_link" />
+    <origin xyz="0 0 0" rpy="-${pi/2} ${pi} 0" />
+    <axis xyz="0 0 1" />
+  </joint>
   <joint name="waist" type="revolute" >
     <parent link="base_link" />
@@ -115,5 +124,5 @@
     <parent link="tip" />
     <child link="stylus" />
-    <origin xyz="0 -0.023 0" rpy="3.14159 3.14159 0" />
+    <origin xyz="0 -0.023 0" rpy="${pi} ${pi} 0" />
     <axis xyz="0 1 0" />
     <limit lower="-2.58" upper="2.58" velocity="100" effort="5" />
